File: hardware/esp32-eter.kicad_sch (KiCad schematic)
At the start: 41 parts, among them J1 USB_C_Receptacle_USB2.0, J2 Conn_01x15_Pin, J3 Conn_01x15_Pin, SW1 BOOT, SW2 EN, U1 ESP32-WROOM-32, U2 USBLC6-2SC6, U3 CP2102N-Axx-xQFN28, U4 TLV76733DRVx, U5 BME280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

Commit message: PROJECT-ETHER-MAIN: Change the resistor value for the led diode.
Parts:
- R9: value 1k -> 330
Changed lines of the file:
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@@
       (effects (font (size 1.27 1.27)) (justify left))
     )
-    (property "Value" "1k" (at 90.17 148.59 0)
+    (property "Value" "330" (at 90.17 148.59 0)
       (effects (font (size 1.27 1.27)) (justify left))
     )
